File: pcb/Video-Frame.kicad_pcb (KiCad board)
At the start: 0 parts

Commit message: PCB Layout
Changes in schematic
+ Fixed +3V3_SD Power NET
+ Changed 100uF electrolytic to 10uF tantalum (lower leakage current)
Parts:
- added C1: 2.2u, Capacitor_SMD:C_0603_1608Metric, F.Cu at (146.8, 109.8)
- added C10: 100n, Capacitor_SMD:C_0603_1608Metric, F.Cu at (148.2, 78.5)
- added C11: 2.2u, Capacitor_SMD:C_0603_1608Metric, F.Cu at (157.8, 78.5)
- added C12: 10u, Capacitor_Tantalum_SMD:CP_EIA-3216-10_Kemet-I, F.Cu at (160.2, 79.2)
- added C13: 15p, Capacitor_SMD:C_0603_1608Metric, F.Cu at (146.8, 88.2)
- added C14: 2.2u, Capacitor_SMD:C_0603_1608Metric, F.Cu at (98.5, 102.5)
- added C15: 15p, Capacitor_SMD:C_0603_1608Metric, F.Cu at (149.0, 88.2)
- added C16: 100n, Capacitor_SMD:C_0603_1608Metric, F.Cu at (121.5, 113.4)
- added C17: 100n, Capacitor_SMD:C_0603_1608Metric, F.Cu at (121.0, 82.8)
- added C18: 2.2u, Capacitor_SMD:C_0603_1608Metric, F.Cu at (128.2, 97.2)
- added C19: 10u, Capacitor_Tantalum_SMD:CP_EIA-3216-10_Kemet-I, F.Cu at (121.8, 89.7)
- added C2: 100n, Capacitor_SMD:C_0603_1608Metric, F.Cu at (126.8, 110.5)
- added C20: 10u, Capacitor_Tantalum_SMD:CP_EIA-3216-10_Kemet-I, F.Cu at (127.8, 89.8)
- added C21: 2.2u, Capacitor_SMD:C_0603_1608Metric, F.Cu at (147.5, 112.8)
- added C22: 2.2u, Capacitor_SMD:C_0603_1608Metric, F.Cu at (106.0, 93.0)
- added C23: 100n, Capacitor_SMD:C_0603_1608Metric, F.Cu at (147.0, 119.0)
- added C24: 2.2u, Capacitor_SMD:C_0603_1608Metric, F.Cu at (144.8, 102.2)
- added C25: 2.2u, Capacitor_SMD:C_0603_1608Metric, F.Cu at (131.8, 96.8)
- added C26: 15p, Capacitor_SMD:C_0603_1608Metric, F.Cu at (137.8, 122.0)
- added C27: 15p, Capacitor_SMD:C_0603_1608Metric, F.Cu at (141.0, 122.0)
- added C28: 15p, Capacitor_SMD:C_0603_1608Metric, F.Cu at (130.8, 122.8)
- added C29: 15p, Capacitor_SMD:C_0603_1608Metric, F.Cu at (133.2, 122.8)
- added C3: 100n, Capacitor_SMD:C_0603_1608Metric, F.Cu at (138.2, 114.5)
- added C30: 10u, Capacitor_Tantalum_SMD:CP_EIA-3216-10_Kemet-I, F.Cu at (124.8, 89.8)
- added C4: 100n, Capacitor_SMD:C_0603_1608Metric, F.Cu at (143.8, 109.8)
- added C5: 100n, Capacitor_SMD:C_0603_1608Metric, F.Cu at (144.8, 100.5)
- added C6: 100n, Capacitor_SMD:C_0603_1608Metric, F.Cu at (128.2, 99.5)
- added C7: 100n, Capacitor_SMD:C_0603_1608Metric, F.Cu at (129.8, 114.2)
- added C8: 10u, Capacitor_Tantalum_SMD:CP_EIA-3216-10_Kemet-I, F.Cu at (141.2, 82.0)
- added C9: 2.2u, Capacitor_SMD:C_0603_1608Metric, F.Cu at (144.2, 82.2)
- added D1: SS14, Diode_SMD:D_SMA, F.Cu at (112.0, 79.5)
- added D2: SS14, Diode_SMD:D_SMA, F.Cu at (153.2, 78.0)
- added D3: SS14, Diode_SMD:D_SMA, F.Cu at (112.0, 87.0)
- added D4: SS14, Diode_SMD:D_SMA, F.Cu at (125.2, 79.5)
- added F1: 500mA, Fuse:Fuse_1812_4532Metric, F.Cu at (106.2, 79.0)
- added F2: 500mA, Fuse:Fuse_1812_4532Metric, F.Cu at (106.8, 88.8)
- added J1: POWER, Connector_PinHeader_2.54mm:PinHeader_1x02_P2.54mm_Vertical, F.Cu at (98.0, 85.0)
- added J2: USB_B_Micro, Connector_MicroUSB:USB_Micro-B_CUI_Devices-UJ2-MIBH-G-SMT-TR, F.Cu at (97.2, 94.8)
- added J3: DBG_SWD, Connector_PinHeader_2.54mm:PinHeader_1x06_P2.54mm_Vertical, F.Cu at (112.3, 122.0)
- added J4: Micro_SD_Card_Det, Connector_Card:microSD_HC_Molex_104031-0811, F.Cu at (101.5, 110.5)
- added J5: DISPLAY, Connector_PinHeader_2.54mm:PinHeader_1x08_P2.54mm_Horizontal, B.Cu at (172.0, 97.0)
- added J6: USART3, Connector_PinHeader_2.54mm:PinHeader_1x03_P2.54mm_Vertical, F.Cu at (172.0, 86.0)
- added L1: MWSA0402S-4R7MT, Inductor_SMD:L_Murata_LQH55DN_5.7x5.0mm, F.Cu at (154.2, 83.0)
- added R1: 0Ω, Resistor_SMD:R_0603_1608Metric, F.Cu at (128.5, 78.0)
- added R10: LDR, OptoDevice:R_LDR_5.1x4.3mm_P3.4mm_Vertical, F.Cu at (117.0, 111.0)
- added R11: 33KΩ, Resistor_SMD:R_0603_1608Metric, F.Cu at (136.5, 88.6)
- added R12: 33KΩ, Resistor_SMD:R_0603_1608Metric, F.Cu at (136.4, 92.0)
- added R13: 100Ω, Resistor_SMD:R_0603_1608Metric, F.Cu at (121.5, 111.4)
- added R14: 0Ω, Resistor_SMD:R_0603_1608Metric, F.Cu at (116.0, 77.5)
- added R16: 1MΩ, Resistor_SMD:R_0603_1608Metric, F.Cu at (115.5, 88.8)
- added R17: 1MΩ, Resistor_SMD:R_0603_1608Metric, F.Cu at (115.5, 85.2)
- added R18: 1MΩ, Resistor_SMD:R_0603_1608Metric, F.Cu at (115.5, 81.8)
- added R19: 100Ω, Resistor_SMD:R_0603_1608Metric, F.Cu at (114.0, 118.0)
- added R2: 33KΩ, Resistor_SMD:R_0603_1608Metric, F.Cu at (132.1, 80.8)
- added R20: 100Ω, Resistor_SMD:R_0603_1608Metric, F.Cu at (116.0, 118.0)
- added R21: 100Ω, Resistor_SMD:R_0603_1608Metric, F.Cu at (143.0, 112.8)
- added R22: 100Ω, Resistor_SMD:R_0603_1608Metric, F.Cu at (122.0, 118.0)
- added R23: 100Ω, Resistor_SMD:R_0603_1608Metric, F.Cu at (144.8, 122.8)
- added R24: 1MΩ, Resistor_SMD:R_0603_1608Metric, F.Cu at (114.8, 92.0)
- added R25: 100Ω, Resistor_SMD:R_0603_1608Metric, F.Cu at (124.0, 118.0)
- added R26: 100Ω, Resistor_SMD:R_0603_1608Metric, F.Cu at (126.0, 118.0)
- added R27: 33KΩ, Resistor_SMD:R_0603_1608Metric, F.Cu at (147.0, 122.8)
- added R28: 33KΩ, Resistor_SMD:R_0603_1608Metric, F.Cu at (106.0, 100.8)
- added R29: 33KΩ, Resistor_SMD:R_0603_1608Metric, F.Cu at (109.2, 100.0)
- added R3: 33KΩ, Resistor_SMD:R_0603_1608Metric, F.Cu at (159.3, 87.5)
- added R30: 100Ω, Resistor_SMD:R_0603_1608Metric, F.Cu at (110.5, 114.5)
- added R31: 100Ω, Resistor_SMD:R_0603_1608Metric, F.Cu at (110.5, 112.0)
- added R32: 100Ω, Resistor_SMD:R_0603_1608Metric, F.Cu at (135.2, 116.2)
- added R33: 0Ω, Resistor_SMD:R_0603_1608Metric, F.Cu at (166.5, 96.2)
- added R34: 100Ω, Resistor_SMD:R_0603_1608Metric, F.Cu at (110.5, 110.0)
- added R35: 33KΩ, Resistor_SMD:R_0603_1608Metric, F.Cu at (111.2, 100.0)
- added R36: 100Ω, Resistor_SMD:R_0603_1608Metric, F.Cu at (165.2, 102.0)
- added R37: 100Ω, Resistor_SMD:R_0603_1608Metric, F.Cu at (110.5, 108.0)
- added R38: 100Ω, Resistor_SMD:R_0603_1608Metric, F.Cu at (165.8, 104.5)
- added R39: 100Ω, Resistor_SMD:R_0603_1608Metric, F.Cu at (165.8, 107.0)
- added R4: 33KΩ, Resistor_SMD:R_0603_1608Metric, F.Cu at (134.6, 81.5)
- added R40: 100Ω, Resistor_SMD:R_0603_1608Metric, F.Cu at (110.5, 105.5)
- added R41: 100Ω, Resistor_SMD:R_0603_1608Metric, F.Cu at (165.8, 109.5)
- added R42: 100Ω, Resistor_SMD:R_0603_1608Metric, F.Cu at (110.5, 103.5)
- added R43: 100Ω, Resistor_SMD:R_0603_1608Metric, F.Cu at (165.8, 112.0)
- added R44: 100Ω, Resistor_SMD:R_0603_1608Metric, F.Cu at (110.5, 116.5)
- added R45: 100Ω, Resistor_SMD:R_0603_1608Metric, F.Cu at (164.5, 114.8)
- added R46: 33KΩ, Resistor_SMD:R_0603_1608Metric, F.Cu at (165.3, 99.5)
- added R47: 100Ω, Resistor_SMD:R_0603_1608Metric, F.Cu at (166.0, 91.0)
- added R48: 100Ω, Resistor_SMD:R_0603_1608Metric, F.Cu at (166.0, 88.5)
- added R49: 100Ω, Resistor_SMD:R_0603_1608Metric, F.Cu at (133.2, 116.2)
- added R5: 33KΩ, Resistor_SMD:R_0603_1608Metric, F.Cu at (155.6, 87.5)
- added R6: 33KΩ, Resistor_SMD:R_0603_1608Metric, F.Cu at (145.0, 88.2)
- added R7: 33KΩ, Resistor_SMD:R_0603_1608Metric, F.Cu at (152.0, 87.5)
- added R8: 0Ω, Resistor_SMD:R_0603_1608Metric, F.Cu at (141.5, 87.4)
- added R9: 33KΩ, Resistor_SMD:R_0603_1608Metric, F.Cu at (103.2, 102.5)
- added SW1: BOOT, Button_Switch_THT:SW_PUSH_6mm, F.Cu at (166.0, 123.0)
- added SW2: RESET, Button_Switch_THT:SW_PUSH_6mm, F.Cu at (156.0, 123.0)
- added TP1: PA1, TestPoint:TestPoint_Pad_D1.0mm, F.Cu at (157.2, 112.0)
- added TP10: PC2, TestPoint:TestPoint_Pad_D1.0mm, F.Cu at (151.0, 115.0)
- added TP11: PC3, TestPoint:TestPoint_Pad_D1.0mm, F.Cu at (160.2, 115.0)
- added TP12: PB5, TestPoint:TestPoint_Pad_D1.0mm, F.Cu at (122.0, 105.0)
- added TP13: PC6, TestPoint:TestPoint_Pad_D1.0mm, F.Cu at (160.0, 94.0)
- added TP14: PB6, TestPoint:TestPoint_Pad_D1.0mm, F.Cu at (119.0, 108.0)
- added TP15: PC7, TestPoint:TestPoint_Pad_D1.0mm, F.Cu at (157.0, 94.0)
- added TP16: PB7, TestPoint:TestPoint_Pad_D1.0mm, F.Cu at (122.0, 108.0)
- added TP17: PC13, TestPoint:TestPoint_Pad_D1.0mm, F.Cu at (154.2, 115.0)
- added TP18: PB13, TestPoint:TestPoint_Pad_D1.0mm, F.Cu at (160.0, 98.0)
- added TP19: PB14, TestPoint:TestPoint_Pad_D1.0mm, F.Cu at (157.0, 98.0)
- added TP2: PA2, TestPoint:TestPoint_Pad_D1.0mm, F.Cu at (154.2, 112.0)
- added TP20: PB15, TestPoint:TestPoint_Pad_D1.0mm, F.Cu at (154.0, 98.0)
- added TP3: PA3, TestPoint:TestPoint_Pad_D1.0mm, F.Cu at (154.0, 109.0)
- added TP4: PA4, TestPoint:TestPoint_Pad_D1.0mm, F.Cu at (157.0, 109.0)
- added TP5: PA6, TestPoint:TestPoint_Pad_D1.0mm, F.Cu at (160.0, 109.0)
- added TP6: PA8, TestPoint:TestPoint_Pad_D1.0mm, F.Cu at (154.2, 94.0)
- added TP7: PA10, TestPoint:TestPoint_Pad_D1.0mm, F.Cu at (151.2, 94.0)
- added TP8: PC0, TestPoint:TestPoint_Pad_D1.0mm, F.Cu at (157.2, 115.0)
- added TP9: PC1, TestPoint:TestPoint_Pad_D1.0mm, F.Cu at (160.2, 112.0)
- added U1: MP2451DT, Package_TO_SOT_SMD:SOT-23-6_Handsoldering, F.Cu at (147.2, 83.0)
- added U2: SY6280A, Package_TO_SOT_SMD:SOT-23-5_HandSoldering, F.Cu at (132.8, 77.8)
- added U3: SY6280A, Package_TO_SOT_SMD:SOT-23-5_HandSoldering, F.Cu at (139.5, 91.0)
- added U4: HT7533-1, Package_TO_SOT_SMD:SOT-89-3, F.Cu at (120.2, 79.2)
- added U5: USBLC6-2SC6, Package_TO_SOT_SMD:SOT-23-6, F.Cu at (106.0, 96.0)
- added U6: STM32F405RGT6, Package_QFP:LQFP-64_10x10mm_P0.5mm, F.Cu at (135.2, 106.0)
- added Y1: 8MHz, Crystal:Crystal_SMD_5032-2Pin_5.0x3.2mm, F.Cu at (139.5, 119.0)
- added Y2: 32.768KHz, Crystal:Crystal_SMD_3215-2Pin_3.2x1.5mm, F.Cu at (132.2, 119.8)
Routing:
- net GND: track 0.00 -> 98.4 mm, vias 0 -> 82
- net +3V3_SD: track 0.00 -> 76.0 mm, vias 0 -> 3
- net /3V3_EN: track 0.00 -> 72.2 mm, vias 0 -> 2
- net VDD: track 0.00 -> 53.2 mm, vias 0 -> 11
- net Net-(C21-Pad1): track 0.00 -> 51.3 mm, vias 0 -> 2
- net +BATT: track 0.00 -> 47.4 mm
- net /NRST: track 0.00 -> 42.2 mm, vias 0 -> 2
- net /EP_BUSY: track 0.00 -> 41.8 mm, vias 0 -> 2
- net +3V3: track 0.00 -> 39.5 mm, vias 0 -> 7
- net /USB_VBUS: track 0.00 -> 38.2 mm, vias 0 -> 2
- net /UART3_RX: track 0.00 -> 37.2 mm
- net Net-(TP17-Pad1): track 0.00 -> 35.6 mm, vias 0 -> 2
- net Net-(TP9-Pad1): track 0.00 -> 35.5 mm, vias 0 -> 2
- net /USB_D-: track 0.00 -> 33.6 mm
- net /USB_D+: track 0.00 -> 33.5 mm
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- added copper zone on F.Cu, net +3V3
- added copper zone on In2.Cu, net +3V3
- added copper zone on B.Cu, net GND
- added copper zone on F.Cu, net GND
- added copper zone on In1.Cu, net GND
- added copper zone on F.Cu, net Net-(C10-Pad1)
- added copper zone on In2.Cu, net VDD
Other:
- board outline added: 80 x 50 mm
- copper layers 0 -> 4
- board text added: "+"
- board text added: "+3V3"
- board text added: "+4V/+12V"
- board text added: "BUSY"
- board text added: "CLK"
- board text added: "CS"
- board text added: "DC"
- board text added: "DISPLAY"
- board text added: "GND"
- board text added: "JLCJLCJLCJLC"
- board text added: "MOSI"
- board text added: "NRST"
- board text added: "POWER"
- board text added: "RST"
- board text added: "RX"
- board text added: "SWCLK"
- board text added: "SWD"
- board text added: "SWDIO"
- board text added: "SWO"
- board text added: "TX"
- board text added: "UART3"
- board text added: "VDD"
- board text added: "Video Frame revA ts-manuel 02/2021"
- board text added: "https://github.com/ts-manuel/VideoFrame"
